Commit message: add box stacking env, todo: finish pseudolikelihood and add rotation

File: ebor/Envs/Assets/cube_blue.urdf (robot description, URDF)
Before this commit: robot cube.urdf, 1 links, 0 joints
Links:
- link baseLink: geometry collision box size=.07 .07 .07; visual mesh filename=cube.obj scale=.07 .07 .07

File: ebor/Envs/Assets/cube_green.urdf (robot description, URDF)
Before this commit: robot cube.urdf, 1 links, 0 joints
Links:
- link baseLink: geometry collision box size=.07 .07 .07; visual mesh filename=cube.obj scale=.07 .07 .07

File: ebor/Envs/Assets/cube_red.urdf (robot description, URDF)
Before this commit: robot cube.urdf, 1 links, 0 joints
Links:
- link baseLink: geometry collision box size=.07 .07 .07; visual mesh filename=cube.obj scale=.07 .07 .07
